Commit message: update max

File: resources/robots/max/urdf/max.urdf (robot description, URDF)
Before this commit: robot x_leopard, 23 links, 22 joints
Links:
- link body: geometry collision box size=0.283 0.205 0.11; visual mesh filename=../meshes/visual/body.dae
- link link_FL1: geometry collision cylinder length=0.0255 radius=0.047; visual mesh filename=../meshes/visual/link_FL1.STL
- link link_FL2: geometry collision box size=0.2 0.025 0.035; collision cylinder length=0.025 radius=0.023
- link link_FL3: geometry collision box size=0.24 0.02 0.018; visual mesh filename=../meshes/visual/link_FL3.STL
- link link_FLW: geometry collision cylinder length=0.012 radius=0.028; visual mesh filename=../meshes/visual/link_FLW.STL
- link link_FR1: geometry collision cylinder length=0.0255 radius=0.047; visual mesh filename=../meshes/visual/link_FR1.STL
- link link_FR2: geometry collision box size=0.2 0.025 0.035; collision cylinder length=0.025 radius=0.023
- link link_FR3: geometry collision box size=0.24 0.02 0.018; visual mesh filename=../meshes/visual/link_FR3.STL
- link link_FRW: geometry collision cylinder length=0.012 radius=0.028; visual mesh filename=../meshes/visual/link_FRW.STL
- link link_HL1: geometry collision cylinder length=0.0255 radius=0.047; visual mesh filename=../meshes/visual/link_HL1.STL
- link link_HL2: geometry collision box size=0.2 0.025 0.035; collision cylinder length=0.025 radius=0.023
- link link_HL3: geometry collision box size=0.24 0.02 0.018; visual mesh filename=../meshes/visual/link_HL3.STL
- link link_HLW: geometry collision cylinder length=0.016 radius=0.036; visual mesh filename=../meshes/visual/link_HLW.STL
- link link_HR1: geometry collision cylinder length=0.0255 radius=0.047; visual mesh filename=../meshes/visual/link_HR1.STL
- link link_HR2: geometry collision box size=0.2 0.025 0.035; collision cylinder length=0.025 radius=0.023
- link link_HR3: geometry collision box size=0.24 0.02 0.018; visual mesh filename=../meshes/visual/link_HR3.STL
- link link_HRW: geometry collision cylinder length=0.016 radius=0.036; visual mesh filename=../meshes/visual/link_HRW.STL

File: resources/robots/max/urdf/max_ext.urdf (robot description, URDF)
Before this commit: robot max, 23 links, 22 joints
Links:
- link body: geometry collision box size=0.28300 0.20500 0.11000; visual mesh filename=../meshes/visual/body.dae
