Commit message: update aliengo

File: resources/robots/aliengo/aliengo.urdf (robot description, URDF)
Before this commit: robot aliengo_description, 18 links, 17 joints
Joints:
- joint FL_upper_joint: type continuous -> revolute
- joint FR_upper_joint: type continuous -> revolute
- joint RL_upper_joint: type continuous -> revolute
- joint RR_upper_joint: type continuous -> revolute
