Commit message: update laikago

File: resources/robots/laikago/laikago_toes_zup.urdf (robot description, URDF)
Before this commit: robot plane, 17 links, 16 joints
Joints:
- joint FL_hip_motor_2_chassis_joint: type continuous -> revolute
- joint FL_lower_leg_2_upper_leg_joint: type continuous -> revolute
- joint FL_upper_leg_2_hip_motor_joint: type continuous -> revolute
- joint FR_hip_motor_2_chassis_joint: type continuous -> revolute
- joint FR_lower_leg_2_upper_leg_joint: type continuous -> revolute
- joint FR_upper_leg_2_hip_motor_joint: type continuous -> revolute
- joint RL_hip_motor_2_chassis_joint: type continuous -> revolute
- joint RL_lower_leg_2_upper_leg_joint: type continuous -> revolute
- joint RL_upper_leg_2_hip_motor_joint: type continuous -> revolute
- joint RR_hip_motor_2_chassis_joint: type continuous -> revolute
- joint RR_lower_leg_2_upper_leg_joint: type continuous -> revolute
- joint RR_upper_leg_2_hip_motor_joint: type continuous -> revolute
