Commit message: update cheetah urdf

File: resources/robots/cheetah/mini_cheetah.urdf (robot description, URDF)
Before this commit: robot mini_cheetah, 17 links, 16 joints
Joints:
- joint abduct_fl_to_thigh_fl_j: limit (none) -> lower=-4.3633 upper=1.2217 effort=18 velocity=20
- joint abduct_fr_to_thigh_fr_j: limit (none) -> lower=-4.3633 upper=1.2217 effort=18 velocity=20
- joint abduct_hl_to_thigh_hl_j: limit (none) -> lower=-4.3633 upper=1.2217 effort=18 velocity=20
- joint abduct_hr_to_thigh_hr_j: limit (none) -> lower=-4.3633 upper=1.2217 effort=18 velocity=20
- joint thigh_fl_to_knee_fl_j: limit (none) -> lower=-2.4496 upper=2.5440 effort=18 velocity=33
- joint thigh_fr_to_knee_fr_j: limit (none) -> lower=-2.4496 upper=2.5440 effort=18 velocity=33
- joint thigh_hl_to_knee_hl_j: limit (none) -> lower=-2.3995 upper=2.5855 effort=18 velocity=33
- joint thigh_hr_to_knee_hr_j: limit (none) -> lower=-2.3995 upper=2.5855 effort=18 velocity=33
- joint torso_to_abduct_fl_j: limit (none) -> lower=-0.697 upper=0.872 effort=18 velocity=20
- joint torso_to_abduct_fr_j: limit (none) -> lower=-0.872 upper=0.697 effort=18 velocity=20
- joint torso_to_abduct_hl_j: limit (none) -> lower=-0.697 upper=0.872 effort=18 velocity=20
- joint torso_to_abduct_hr_j: limit (none) -> lower=-0.872 upper=0.697 effort=18 velocity=20
